File: single band active eq/SingleBandParametricEQ.kicad_sch (KiCad schematic)
At the start: 18 parts, among them U1 TL081, U2 TL084

Commit message: Added Powering Section
Parts:
- added C3: C_Polarized_US, symbol Device:C_Polarized_US
- added R10, R12: R, symbol Device:R
Connections:
- net -9V is gone; now on net GND: U1.4 (V-), U2.11 (V-)
- net GND: now also C3.2, R12.2; no longer U1.3 (+), U2.10 (+), U2.12 (+), U2.3 (+), U2.5 (+)
- net +9V renamed VCC
- net VCC: now also R10.1
- new net VREF: C3.1, R10.2, R12.1, U1.3 (+), U2.10 (+), U2.12 (+), U2.3 (+), U2.5 (+)
Other:
- note added: "Op Amp Power"
- note added: "Supply Splitting"
- note removed: "Power"
